File: CareLoop/max30102.kicad_sch (KiCad schematic)
At the start: 16 parts, among them U1 MCP1700x-180xxMB, U2 MAX30102, U7 PCA9306

Commit message: update PCB
Parts:
- C20, C25, C27: JLCPCB Part#(optional) (none) -> C161494
- C21, C23: JLCPCB Part#(optional) (none) -> C1538
- C22: JLCPCB Part#(optional) (none) -> C88945
- C24: JLCPCB Part#(optional) (none) -> C15525
- C26: JLCPCB Part#(optional) (none) -> C62550
- JP1_MAX30102: footprint Connector_PinHeader_1.00mm:PinHeader_1x02_P1.00mm_Vertical -> Connector_PinHeader_2.00mm:PinHeader_1x02_P2.00mm_Vertical; now not fitted
- R20: JLCPCB Part#(optional) (none) -> C25531
- R21: JLCPCB Part#(optional) (none) -> C22369193
- R22, R23: JLCPCB Part#(optional) (none) -> C22369185
- U1: JLCPCB Part#(optional) (none) -> C631991
- U2: JLCPCB Part#(optional) (none) -> C6454833
- U7: JLCPCB Part#(optional) (none) -> C33196
Changed lines of the file:
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@@
+			)
+		)
+		(property "JLCPCB Part#(optional)" "C631991"
+			(at 138.43 76.2 90)
+			(effects
+				(font
+					(size 1.27 1.27)
+				)
+				(hide yes)
 			)
 		)
@@
 		(in_bom yes)
 		(on_board yes)
-		(dnp no)
+		(dnp yes)
 		(fields_autoplaced yes)
 		(property "Reference" "JP1_MAX30102"
@@
 			)
 		)
-		(property "Footprint" "Connector_PinHeader_1.00mm:PinHeader_1x02_P1.00mm_Vertical"
+		(property "Footprint" "Connector_PinHeader_2.00mm:PinHeader_1x02_P2.00mm_Vertical"
 			(at 138.43 44.45 0)
 			(effects
@@
 			)
 		)
+		(property "JLCPCB Part#(optional)" ""
+			(at 138.43 44.45 90)
+			(effects
+				(font
+					(size 1.27 1.27)
+				)
+				(hide yes)
+			)
+		)
 		(pin "1"
 		)
@@
 			)
 		)
+		(property "JLCPCB Part#(optional)" "C161494"
+			(at 107.95 60.96 0)
+			(effects
+				(font
+					(size 1.27 1.27)
+				)
+				(hide yes)
+			)
+		)
 		(pin "1"
 		)
@@
 			)
 		)
+		(property "JLCPCB Part#(optional)" "C22369193"
+			(at 67.31 133.35 0)
+			(effects
+				(font
+					(size 1.27 1.27)
+				)
+				(hide yes)
+			)
+		)
 		(pin "2"
 		)
@@
 			)
 		)
+		(property "JLCPCB Part#(optional)" "C33196"
+			(at 85.09 109.22 0)
+			(effects
+				(font
+					(size 1.27 1.27)
+				)
+				(hide yes)
+			)
+		)
 		(pin "8"
 		)
@@
 			)
 		)
+		(property "JLCPCB Part#(optional)" "C161494"
+			(at 168.91 91.44 0)
+			(effects
+				(font
+					(size 1.27 1.27)
+				)
+				(hide yes)
+			)
+		)
 		(pin "1"
 		)
@@
 			)
 		)
+		(property "JLCPCB Part#(optional)" "C6454833"
+			(at 143.51 109.22 0)
+			(effects
+				(font
+					(size 1.27 1.27)
+				)
+				(hide yes)
+			)
+		)
 		(pin "3"
 		)
@@
 			)
 		)
+		(property "JLCPCB Part#(optional)" "C22369185"
+			(at 106.68 99.06 0)
+			(effects
+				(font
+					(size 1.27 1.27)
+				)
+				(hide yes)
+			)
+		)
 		(pin "2"
 		)
@@
 			)
 		)
+		(property "JLCPCB Part#(optional)" "C15525"
+			(at 156.21 91.44 0)
+			(effects
+				(font
+					(size 1.27 1.27)
+				)
+				(hide yes)
+			)
+		)
 		(pin "1"
 		)
@@
 			)
 		)
+		(property "JLCPCB Part#(optional)" "C22369185"
+			(at 110.49 99.06 0)
+			(effects
+				(font
+					(size 1.27 1.27)
+				)
+				(hide yes)
+			)
+		)
 		(pin "2"
 		)
@@
 			)
 		)
+		(property "JLCPCB Part#(optional)" "C161494"
+			(at 52.07 106.68 0)
+			(effects
+				(font
+					(size 1.27 1.27)
+				)
+				(hide yes)
+			)
+		)
 		(pin "2"
 		)
@@
 			)
 		)
+		(property "JLCPCB Part#(optional)" "C1538"
+			(at 118.11 60.96 0)
+			(effects
+				(font
+					(size 1.27 1.27)
+				)
+				(hide yes)
+			)
+		)
 		(pin "1"
 		)
@@
 			)
 		)
+		(property "JLCPCB Part#(optional)" "C62550"
+			(at 43.18 106.68 0)
+			(effects
+				(font
+					(size 1.27 1.27)
+				)
+				(hide yes)
+			)
+		)
 		(pin "2"
 		)
@@
 			)
 		)
+		(property "JLCPCB Part#(optional)" "C1538"
+			(at 129.54 95.25 0)
+			(effects
+				(font
+					(size 1.27 1.27)
+				)
+				(hide yes)
+			)
+		)
 		(pin "1"
 		)
@@
 			)
 		)
+		(property "JLCPCB Part#(optional)" "C88945"
+			(at 118.11 95.25 0)
+			(effects
+				(font
+					(size 1.27 1.27)
+				)
+				(hide yes)
+			)
+		)
 		(pin "1"
 		)
@@
 			(at 179.07 99.06 0)
 			(effects
+				(font
+					(size 1.27 1.27)
+				)
+				(hide yes)
+			)
+		)
+		(property "JLCPCB Part#(optional)" "C25531"
+			(at 179.07 99.06 0)
+			(effects

Commit message: nordic review
Parts:
- C20, C25, C27: JLCPCB Part#(optional) C161494 -> C161404
Changed lines of the file:
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@@
 			)
 		)
-		(property "JLCPCB Part#(optional)" "C161494"
+		(property "JLCPCB Part#(optional)" "C161404"
 			(at 107.95 60.96 0)
 			(effects
@@
 			)
 		)
-		(property "JLCPCB Part#(optional)" "C161494"
+		(property "JLCPCB Part#(optional)" "C161404"
 			(at 168.91 91.44 0)
 			(effects
@@
 			)
 		)
-		(property "JLCPCB Part#(optional)" "C161494"
+		(property "JLCPCB Part#(optional)" "C161404"
 			(at 52.07 106.68 0)
 			(effects
